Commit message: adding slam

File: pet_bot_test5/urdf/pet_bot_test5.urdf.xacro (robot description, xacro)
@@ -1037,3 +1037,28 @@
     <origin xyz="0.003 -0.13 0.030" rpy="0 0 -1.57"/>
   </joint>
+ <link name="imu_link">
+ <visual>
+      <geometry>
+        <box size="0.02 0.02 0.005"/>
+      </geometry>
+      <material name="imu_color">
+        <color rgba="1.0 0.2 0.0 1.0"/>
+      </material>
+    </visual>
+    <collision>
+      <geometry>
+        <box size="0.02 0.02 0.005"/>
+      </geometry>
+    </collision>
+    <inertial>
+      <mass value="0.001"/>
+      <origin xyz="0 0 0" rpy="0 0 0"/>
+      <inertia ixx="1e-7" ixy="0" ixz="0" iyy="1e-7" iyz="0" izz="1e-7"/>
+    </inertial>
+  </link>
+ <joint name="imu_joint" type="fixed">
+  <parent link="base_link"/>
+  <child link="imu_link"/>
+  <origin xyz="0 0 0" rpy="0 0 0"/>
+</joint>
 </robot>

File: pet_bot_test5/urdf/ros2_control.xacro (robot description, xacro)
@@ -227,3 +227,12 @@
     </plugin>
   </gazebo>
+  <!-- ========================================================= -->
+  <!--                    IMU PLUGIN                   -->
+  <!-- ========================================================= -->
+<gazebo>
+<plugin
+    filename="libignition-gazebo-imu-system.so"
+    name="ignition::gazebo::systems::Imu">
+  </plugin>
+  </gazebo>
 </robot>

File: pet_bot_test5/urdf/sensors.xacro (robot description, xacro)
@@ -57,3 +57,27 @@
     </sensor>
   </gazebo>
-</robot>
+  <!-- ========================================================= -->
+  <!--                         IMU                               -->
+  <!-- ========================================================= -->
+  <gazebo reference ="imu_link">
+  <sensor name="imu_sensor" type="imu">
+      <always_on>true</always_on>
+      <update_rate>100</update_rate>
+      <visualize>true</visualize>
+      <topic>imu</topic>
+      <gz_frame_id>imu_link</gz_frame_id>
+      <imu>
+        <angular_velocity>
+          <x><noise type="gaussian"><mean>0.0</mean><stddev>2e-4</stddev></noise></x>
+          <y><noise type="gaussian"><mean>0.0</mean><stddev>2e-4</stddev></noise></y>
+          <z><noise type="gaussian"><mean>0.0</mean><stddev>2e-4</stddev></noise></z>
+        </angular_velocity>
+        <linear_acceleration>
+          <x><noise type="gaussian"><mean>0.0</mean><stddev>1.7e-2</stddev></noise></x>
+          <y><noise type="gaussian"><mean>0.0</mean><stddev>1.7e-2</stddev></noise></y>
+          <z><noise type="gaussian"><mean>0.0</mean><stddev>1.7e-2</stddev></noise></z>
+        </linear_acceleration>
+      </imu>
+    </sensor>
+  </gazebo>
+  </robot>
